File: sdo_to_quiic_qt_led.sch (EAGLE design)
At the start: 10 parts

Commit message: saving progress
Parts:
- JP2: device pinhead:PINHD-2X2 -> microbuilder:HEADER-2X3
Connections:
- new net SAO_GPIO1: JP2.1
- new net SAO_GPIO2: JP2.2
- net GND: now also JP2.6; no longer JP2.3
- net SDA: now also JP2.3; no longer JP2.2
- net VCC: now also JP2.5; no longer JP2.1
Other:
- note removed: "SAO Header"
