File: sdo_to_quiic_qt_led.brd (EAGLE design)
At the start: 25.4 x 17.8 mm, 11 parts

Commit message: saving progress
Parts:
- JP2: device pinhead:2X02 -> microbuilder:2X03_ROUND_70MIL
- moved R2 9.23 mm to (7.49, 13.1)
- moved R1 7.60 mm to (11.6, 4.95)
- turned JP2 to 180 degrees
Connections:
- new net SAO_GPIO1: JP2.1
- new net SAO_GPIO2: JP2.2
- net GND: now also JP2.6; no longer JP2.3
- net SDA: now also JP2.3; no longer JP2.2
- net VCC: now also JP2.5; no longer JP2.1
Routing:
- net SDA: track 0.00 -> 41.7 mm
- net VCC: track 0.00 -> 39.1 mm, vias 0 -> 2
- net SCL: track 0.00 -> 26.1 mm
Other:
- board size 25.4 x 17.8 mm -> 25.4 x 47 mm
- board text added: "D0/A4/SDA"
- board text added: "D1/A0/VOUT"
- board text added: "D2/A1/SCL/MISO"
- board text added: "D3/A3/TXD/SCK"
- board text added: "D4/A2/RXD/MOSI"

Commit message: routed
Parts:
- moved R2 4.07 mm to (11.4, 12.1)
Routing:
- net SDA: track 41.7 -> 33.1 mm
- net VCC: track 39.1 -> 35.9 mm, vias 2 -> 1
- net SCL: track 26.1 -> 23.1 mm
Other:
- board size 25.4 x 47 mm -> 25.4 x 17.8 mm
- board text removed: "D0/A4/SDA"
- board text removed: "D1/A0/VOUT"
- board text removed: "D2/A1/SCL/MISO"
- board text removed: "D3/A3/TXD/SCK"
- board text removed: "D4/A2/RXD/MOSI"
- board text removed: "on"
