File: sdo_to_quiic.brd (EAGLE design)
At the start: 25.4 x 17.8 mm, 11 parts

Commit message: renamed, tweaked
Parts:
- moved R1 0.13 mm to (11.4, 4.95)
Changed lines of the file:
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@@
 <attribute name="VALUE" x="7.62" y="-0.635" size="0.4064" layer="27" ratio="10"/>
 </element>
-<element name="R1" library="microbuilder" package="0805-NO" value="10K" x="11.557" y="4.953" smashed="yes">
-<attribute name="NAME" x="8.636" y="4.572" size="0.8128" layer="25" font="vector" ratio="18"/>
-<attribute name="VALUE" x="13.335" y="4.191" size="0.4064" layer="27" font="vector" ratio="10"/>
+<element name="R1" library="microbuilder" package="0805-NO" value="10K" x="11.43" y="4.953" smashed="yes">
+<attribute name="NAME" x="8.509" y="4.572" size="0.8128" layer="25" font="vector" ratio="18"/>
+<attribute name="VALUE" x="13.208" y="4.191" size="0.4064" layer="27" font="vector" ratio="10"/>
 </element>
 <element name="R2" library="microbuilder" package="0805-NO" value="10K" x="11.43" y="12.065" smashed="yes">
@@
 <contactref element="JP2" pad="4"/>
 <wire x1="12.7" y1="7.62" x2="12.7" y2="6.223" width="0.254" layer="1"/>
-<wire x1="12.7" y1="6.223" x2="12.7" y2="5.146" width="0.254" layer="1"/>
-<wire x1="12.7" y1="5.146" x2="12.507" y2="4.953" width="0.254" layer="1"/>
-<wire x1="12.507" y1="4.953" x2="12.507" y2="4.003" width="0.254" layer="1"/>
-<wire x1="12.507" y1="4.003" x2="13.97" y2="2.54" width="0.254" layer="1"/>
+<wire x1="12.7" y1="6.223" x2="12.7" y2="5.273" width="0.254" layer="1"/>
+<wire x1="12.7" y1="5.273" x2="12.38" y2="4.953" width="0.254" layer="1"/>
+<wire x1="12.38" y1="4.953" x2="12.38" y2="4.13" width="0.254" layer="1"/>
+<wire x1="12.38" y1="4.13" x2="13.97" y2="2.54" width="0.254" layer="1"/>
 <wire x1="12.7" y1="8.382" x2="13.208" y2="8.89" width="0.254" layer="1"/>
 <wire x1="12.7" y1="7.62" x2="12.7" y2="8.382" width="0.254" layer="1"/>
@@
 <wire x1="11.303" y1="4.953" x2="8.89" y2="2.54" width="0.3048" layer="16"/>
 <wire x1="11.303" y1="4.953" x2="15.494" y2="4.953" width="0.3048" layer="16"/>
-<wire x1="5.054" y1="9.39" x2="7.993" y2="9.39" width="0.3048" layer="1"/>
-<wire x1="8.763" y1="10.16" x2="7.993" y2="9.39" width="0.3048" layer="1"/>
-<wire x1="10.16" y1="10.16" x2="8.763" y2="10.16" width="0.3048" layer="1"/>
-<wire x1="8.89" y1="2.54" x2="10.607" y2="4.257" width="0.3048" layer="1"/>
-<wire x1="10.607" y1="4.257" x2="10.607" y2="4.953" width="0.3048" layer="1"/>
-<wire x1="10.607" y1="4.953" x2="10.033" y2="4.953" width="0.3048" layer="1"/>
+<wire x1="5.054" y1="9.39" x2="8.628" y2="9.39" width="0.3048" layer="1"/>
+<wire x1="9.398" y1="10.16" x2="8.628" y2="9.39" width="0.3048" layer="1"/>
+<wire x1="10.16" y1="10.16" x2="9.398" y2="10.16" width="0.3048" layer="1"/>
+<wire x1="8.89" y1="2.54" x2="10.48" y2="4.13" width="0.3048" layer="1"/>
+<wire x1="10.48" y1="4.13" x2="10.48" y2="4.953" width="0.3048" layer="1"/>
+<wire x1="10.48" y1="4.953" x2="10.033" y2="4.953" width="0.3048" layer="1"/>
 <wire x1="10.033" y1="4.953" x2="8.382" y2="6.604" width="0.3048" layer="1"/>
 <wire x1="3.556" y1="7.112" x2="4.064" y2="6.604" width="0.3048" layer="1"/>
