File: sdo_to_quiic_qt.brd (EAGLE design)
At the start: 25.4 x 17.8 mm, 11 parts

Commit message: final silk?
Parts:
- moved R1 7.11 mm to (11.4, 12.1)
- moved R2 7.11 mm to (11.4, 4.95)
Connections:
- net SCL: now also R2.2; no longer R1.2
- net SDA: now also R1.2; no longer R2.2
Other:
- board text added: "parturient montes, nascetur ridiculus mus"
- board text removed: "&"
- board text removed: ")"
- board text removed: ","
- board text removed: "O"
- board text removed: "This Is SHITTY"
- board text removed: "VCC MUST BE 3.3V (NO LEVEL SHIFTING)"
- board text removed: "keine erste Wurst, auch keine Extrawurst"
- board text removed: "nein!"
- board text removed: "{"
- board text removed: "|"
Changed lines of the file:
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@@
 <grid distance="0.275" unitdist="mil" unit="mil" style="lines" multiple="1" display="yes" altdistance="1" altunitdist="mil" altunit="mil"/>
 <layers>
-<layer number="1" name="Top" color="4" fill="1" visible="yes" active="yes"/>
+<layer number="1" name="Top" color="4" fill="1" visible="no" active="yes"/>
 <layer number="2" name="Route2" color="1" fill="3" visible="no" active="no"/>
 <layer number="3" name="Route3" color="4" fill="3" visible="no" active="no"/>
@@
 <layer number="20" name="Dimension" color="15" fill="1" visible="no" active="yes"/>
 <layer number="21" name="tPlace" color="14" fill="1" visible="yes" active="yes"/>
-<layer number="22" name="bPlace" color="13" fill="1" visible="yes" active="yes"/>
+<layer number="22" name="bPlace" color="13" fill="1" visible="no" active="yes"/>
 <layer number="23" name="tOrigins" color="14" fill="1" visible="yes" active="yes"/>
 <layer number="24" name="bOrigins" color="13" fill="1" visible="no" active="yes"/>
@@
 <dimension x1="25.4" y1="9.144" x2="0" y2="6.223" x3="12.7" y3="-6.223" textsize="1.778" layer="47" dtype="horizontal" unit="inch"/>
 <dimension x1="13.208" y1="0" x2="12.319" y2="17.78" x3="32.131" y3="8.89" textsize="1.778" layer="47" dtype="vertical" unit="inch"/>
-<text x="16.9418" y="23.5966" size="1.016" layer="22" font="vector" ratio="12" rot="MR0" align="center">This Is
-SHITTY</text>
-<text x="41.6814" y="6.5532" size="1.016" layer="22" font="vector" ratio="12" rot="MR0" align="center">VCC MUST BE 3.3V
-(NO LEVEL SHIFTING)</text>
 <text x="15.367" y="16.637" size="1.016" layer="22" font="vector" ratio="12" rot="MR0" align="center">Revision Mark</text>
 <text x="16.383" y="15.113" size="0.6096" layer="22" font="vector" ratio="12" rot="MR0" align="center">(if this is A,
@@
 <text x="9.93901875" y="16.4084" size="1.778" layer="21" font="vector" ratio="14" align="center">2QUIIC</text>
 <text x="14.89075" y="14.394815625" size="1.778" layer="21" font="vector" ratio="14" align="center">2SHITTY</text>
-<text x="18.792825" y="19.804378125" size="1.778" layer="21" font="vector" ratio="14" align="center">&amp;</text>
 <rectangle x1="16.18425625" y1="13.662659375" x2="16.198225" y2="13.669640625" layer="22" rot="R90"/>
 <rectangle x1="16.1702875" y1="13.655675" x2="16.198225" y2="13.66265625" layer="22" rot="R90"/>
@@
 <rectangle x1="-16.718603125" y1="0.457509375" x2="-16.697653125" y2="0.464490625" layer="200" rot="R90"/>
 <text x="23.553421875" y="4.34466875" size="2.54" layer="22" ratio="15" rot="MR40.3">SO QT!</text>
-<text x="36.873815625" y="18.677890625" size="1.778" layer="22" ratio="15" rot="MR30">O</text>
-<text x="27.6606" y="28.107640625" size="1.778" layer="22" ratio="15" rot="MR30">|</text>
-<text x="29.4836875" y="21.416009375" size="1.778" layer="22" ratio="15" rot="MR30">)</text>
-<text x="32.43135625" y="13.515975" size="1.778" layer="22" ratio="15" rot="MR30">{</text>
 <text x="17.2459625" y="15.59051875" size="0.6096" layer="21" ratio="15" rot="R30">SO QT!</text>
-<text x="16.24710625" y="10.854690625" size="0.6096" layer="21" ratio="15" rot="R43.3">nein!</text>
 <text x="16.289028125" y="9.660253125" size="0.4064" layer="21" ratio="15">keine</text>
 <text x="16.93165" y="9.276075" size="0.4064" layer="21" ratio="15">erste</text>
@@
 <text x="16.631284375" y="6.0140875" size="0.4064" layer="21" ratio="15">keine</text>
 <text x="17.266921875" y="5.51116875" size="0.4064" layer="21" ratio="15">Extrawurst</text>
-<text x="26.473159375" y="-5.0920625" size="0.4064" layer="21" ratio="15">keine erste
-Wurst, auch keine Extrawurst</text>
-<text x="31.977334375" y="10.589259375" size="0.4064" layer="21" ratio="15">erste</text>
-<text x="27.458040625" y="7.348221875" size="0.4064" layer="21" ratio="15">,</text>
-<text x="31.893515625" y="3.82778125" size="0.4064" layer="21" ratio="15">auch</text>
+<text x="12.38758125" y="0.5073625" size="0.6096" layer="22" font="vector" ratio="12" rot="MR0" align="center">parturient montes, nascetur ridiculus mus</text>
 </plain>
 <attributes>
@@
 <attribute name="VALUE" x="7.62" y="-0.635" size="0.4064" layer="27" ratio="10"/>
 </element>
-<element name="R1" library="microbuilder" package="0805-NO" value="10K" x="11.43" y="4.953" smashed="yes">
+<element name="R2" library="microbuilder" package="0805-NO" value="10K" x="11.43" y="4.953" smashed="yes">
 <attribute name="NAME" x="8.509" y="4.572" size="0.8128" layer="25" font="vector" ratio="18"/>
 <attribute name="VALUE" x="13.208" y="4.191" size="0.4064" layer="27" font="vector" ratio="10"/>
 </element>
-<element name="R2" library="microbuilder" package="0805-NO" value="10K" x="11.43" y="12.065" smashed="yes">
+<element name="R1" library="microbuilder" package="0805-NO" value="10K" x="11.43" y="12.065" smashed="yes">
 <attribute name="NAME" x="8.382" y="11.684" size="0.8128" layer="25" font="vector" ratio="18"/>
 <attribute name="VALUE" x="13.208" y="11.303" size="0.4064" layer="27" font="vector" ratio="10"/>
 </element>
 <element name="JP2" library="microbuilder" package="2X03_ROUND_70MIL" value="" x="12.7" y="8.89" smashed="yes" rot="R180">
-<attribute name="NAME" x="12.6492" y="9.3472" size="0.8128" layer="25" ratio="18" rot="R180"/>
 <attribute name="VALUE" x="16.51" y="12.065" size="0.4064" layer="27" ratio="10" rot="R180"/>
 </element>
@@
 <contactref element="CONN1" pad="3"/>
 <contactref element="JP3" pad="4"/>
-<contactref element="R2" pad="2"/>
+<contactref element="R1" pad="2"/>
 <contactref element="JP2" pad="3"/>
 <wire x1="21.59" y1="8.72389375" x2="21.59" y2="6.858" width="0.254" layer="1"/>
@@
 <contactref element="CONN1" pad="4"/>
 <contactref element="JP3" pad="3"/>
-<contactref element="R1" pad="2"/>
+<contactref element="R2" pad="2"/>
 <contactref element="JP2" pad="4"/>
 <wire x1="12.7" y1="7.62" x2="12.7" y2="6.223" width="0.254" layer="1"/>
@@
 <contactref element="CONN2" pad="2"/>
 <contactref element="JP3" pad="1"/>
-<contactref element="R1" pad="1"/>
 <contactref element="R2" pad="1"/>
+<contactref element="R1" pad="1"/>
 <contactref element="JP2" pad="5"/>
 <wire x1="11.303" y1="4.953" x2="8.89" y2="2.54" width="0.3048" layer="16"/>

Commit message: mostly there
Parts:
- removed U$25: (no value), microbuilder:PCBFEAT-REV-040
Routing:
- net VCC: track 35.8 -> 37.4 mm
