File: sdo_to_quiic_qt.brd (EAGLE design)
At the start: 25.4 x 17.8 mm, 10 parts

Commit message: progress
Parts:
- JP2: value (none) -> SAO 1.6 Header
- JP3: value (none) -> Breadboard header
Connections:
- removed net SAO_GPIO1: JP2.1
- removed net SAO_GPIO2: JP2.2
Changed lines of the file:
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@@
 <attribute name="BOM" value="EXCLUDE" x="22.86" y="2.54" size="1.778" layer="27" display="off"/>
 </element>
-<element name="JP3" library="microbuilder" package="1X04_ROUND" value="" x="12.7" y="2.54" smashed="yes">
+<element name="JP3" library="microbuilder" package="1X04_ROUND" value="Breadboard header" x="12.7" y="2.54" smashed="yes">
 <attribute name="VALUE" x="7.62" y="-0.635" size="0.4064" layer="27" ratio="10"/>
 </element>
@@
 <attribute name="VALUE" x="13.208" y="11.303" size="0.4064" layer="27" font="vector" ratio="10"/>
 </element>
-<element name="JP2" library="microbuilder" package="2X03_ROUND_70MIL" value="" x="12.7" y="8.89" smashed="yes" rot="R180">
+<element name="JP2" library="microbuilder" package="2X03_ROUND_70MIL" value="SAO 1.6 Header" x="12.7" y="8.89" smashed="yes" rot="R180">
 <attribute name="VALUE" x="16.51" y="12.065" size="0.4064" layer="27" ratio="10" rot="R180"/>
 </element>
@@
 <wire x1="18.804" y1="8.39" x2="20.346" y2="8.39" width="0.3048" layer="1"/>
 </signal>
-<signal name="SAO_GPIO1">
-<contactref element="JP2" pad="1"/>
-</signal>
-<signal name="SAO_GPIO2">
-<contactref element="JP2" pad="2"/>
-</signal>
 </signals>

Commit message: rearranging
Parts:
- moved R2 0.11 mm to (11.4, 5.06)
Routing:
- net VCC: track 37.4 -> 38.5 mm
Other:
- board text added: "#"
- board text added: "/"
- board text added: "100"
